File: a500hddled.kicad_pcb (KiCad board)
At the start: 2 copper layers, 13.5 x 22.2 mm, 6 parts, among them J1 Male, J2 Female, J3 HDD, Q1 2N3906

Commit message: add 3D models, upgrade kicad
Parts:
- J1: footprint Connector_PinSocket_2.54mm:PinSocket_1x08_P2.54mm_Vertical -> Connector_PinHeader_2.54mm:PinHeader_1x08_P2.54mm_Vertical
- J3: footprint Connector_PinSocket_2.54mm:PinSocket_1x01_P2.54mm_Vertical -> Connector_PinHeader_2.54mm:PinHeader_1x01_P2.54mm_Horizontal
- turned J3 to 90 degrees
Connections:
- J1 pad 5: no_connect_10 -> unconnected-(J1-Pad5)
- J2 pad 5: no_connect_11 -> unconnected-(J2-Pad5)
