File: a500hddled.kicad_sch (KiCad schematic)
At the start: 6 parts, among them J1 Male, J2 Female, J3 HDD, Q1 2N3906

Commit message: add 3D models, upgrade kicad
Parts:
- J1: footprint Connector_PinSocket_2.54mm:PinSocket_1x08_P2.54mm_Vertical -> Connector_PinHeader_2.54mm:PinHeader_1x08_P2.54mm_Vertical
- J3: footprint Connector_PinSocket_2.54mm:PinSocket_1x01_P2.54mm_Vertical -> Connector_PinHeader_2.54mm:PinHeader_1x01_P2.54mm_Horizontal
Changed lines of the file:
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@@
-(kicad_sch (version 20201015) (generator eeschema)
+(kicad_sch (version 20210406) (generator eeschema)
   (paper "A4")
   (junction (at 121.92 50.8) (diameter 1.016) (color 0 0 0 0))
   (junction (at 121.92 60.96) (diameter 1.016) (color 0 0 0 0))
+  (no_connect (at 160.02 60.96))
   (no_connect (at 182.88 60.96))
-  (no_connect (at 160.02 60.96))
   (wire (pts (xy 111.76 60.96) (xy 121.92 60.96))
     (stroke (width 0) (type solid) (color 0 0 0 0))
@@
       (effects (font (size 1.27 1.27)) hide)
     )
+    (pin "1")
   )
   (symbol (lib_id "power:VCC") (at 170.18 55.88 0) (unit 1)
@@
       (effects (font (size 1.27 1.27)) hide)
     )
+    (pin "1")
   )
   (symbol (lib_id "power:VCC") (at 193.04 55.88 0) (unit 1)
@@
       (effects (font (size 1.27 1.27)) hide)
     )
+    (pin "1")
   )
   (symbol (lib_id "power:GND") (at 170.18 66.04 0) (unit 1)
@@
       (effects (font (size 1.27 1.27)) hide)
     )
+    (pin "1")
   )
   (symbol (lib_id "power:GND") (at 193.04 66.04 0) (unit 1)
@@
       (effects (font (size 1.27 1.27)) hide)
     )
+    (pin "1")
   )
   (symbol (lib_id "Device:R_Small") (at 121.92 55.88 0) (unit 1)
@@
       (effects (font (size 1.27 1.27)) hide)
     )
+    (pin "1")
+    (pin "2")
   )
   (symbol (lib_id "Device:R_Small") (at 129.54 60.96 90) (unit 1)
@@
       (effects (font (size 1.27 1.27)) hide)
     )
+    (pin "1")
+    (pin "2")
   )
   (symbol (lib_id "Connector_Generic:Conn_01x01") (at 106.68 60.96 0) (mirror y) (unit 1)
@@
     (property "Reference" "J3" (id 0) (at 108.712 55.4798 0))
     (property "Value" "HDD" (id 1) (at 108.712 57.785 0))
-    (property "Footprint" "Connector_PinSocket_2.54mm:PinSocket_1x01_P2.54mm_Vertical" (id 2) (at 106.68 60.96 0)
+    (property "Footprint" "Connector_PinHeader_2.54mm:PinHeader_1x01_P2.54mm_Horizontal" (id 2) (at 106.68 60.96 0)
       (effects (font (size 1.27 1.27)) hide)
     )
@@
       (effects (font (size 1.27 1.27)) hide)
     )
+    (pin "1")
   )
   (symbol (lib_id "Transistor_BJT:2N3906") (at 137.16 60.96 0) (mirror x) (unit 1)
@@
       (effects (font (size 1.27 1.27)) (justify left) hide)
     )
+    (pin "1")
+    (pin "2")
+    (pin "3")
   )
   (symbol (lib_id "Connector_Generic:Conn_01x08") (at 165.1 58.42 0) (unit 1)
@@
     (property "Reference" "J1" (id 0) (at 164.5921 71.2914 0))
     (property "Value" "Male" (id 1) (at 164.592 73.5838 0))
-    (property "Footprint" "Connector_PinSocket_2.54mm:PinSocket_1x08_P2.54mm_Vertical" (id 2) (at 165.1 58.42 0)
+    (property "Footprint" "Connector_PinHeader_2.54mm:PinHeader_1x08_P2.54mm_Vertical" (id 2) (at 165.1 58.42 0)
       (effects (font (size 1.27 1.27)) hide)
     )
@@
       (effects (font (size 1.27 1.27)) hide)
     )
+    (pin "1")
+    (pin "2")
+    (pin "3")
+    (pin "4")
+    (pin "5")
+    (pin "6")
+    (pin "7")
+    (pin "8")
   )
   (symbol (lib_id "Connector_Generic:Conn_01x08") (at 187.96 58.42 0) (unit 1)
@@
       (effects (font (size 1.27 1.27)) hide)
     )
+    (pin "1")
+    (pin "2")
+    (pin "3")
+    (pin "4")
+    (pin "5")
+    (pin "6")
+    (pin "7")
+    (pin "8")
   )
   (sheet_instances
@@
     )
     (path "/168be580-64bd-4759-bada-531f81446bf9"
-      (reference "J1") (unit 1) (value "Male") (footprint "Connector_PinSocket_2.54mm:PinSocket_1x08_P2.54mm_Vertical")
+      (reference "J1") (unit 1) (value "Male") (footprint "Connector_PinHeader_2.54mm:PinHeader_1x08_P2.54mm_Vertical")
     )
     (path "/9717ba61-b93f-4982-9402-b15a4b7ae6ae"
@@
     )
     (path "/80807bbe-a3e2-4f84-98da-58f11a88ba72"
-      (reference "J3") (unit 1) (value "HDD") (footprint "Connector_PinSocket_2.54mm:PinSocket_1x01_P2.54mm_Vertical")
+      (reference "J3") (unit 1) (value "HDD") (footprint "Connector_PinHeader_2.54mm:PinHeader_1x01_P2.54mm_Horizontal")
     )
     (path "/216a36ed-e222-4c4d-975a-55566d8ec3d4"
